File: BrewGuard PCB/Keyboard/keyboard.kicad_pcb (KiCad board)
At the start: 2 copper layers, 8 parts, among them J1 Tasterplatine, SW1 SW_Push, SW2 SW_Push, SW3 SW_Push

Commit message: corr.
Other:
- board outline added: 38.4 x 30 mm
Changed lines of the file:
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@@
 		)
 		(fill none)
-		(layer "F.Fab")
+		(layer "Edge.Cuts")
 	)
 	(gr_text "BrewGurad KeyPCB"
